File: TeensyIOBreakout.sch (KiCad schematic (older format))
At the start: 1 part

Commit message: SCH and PCB layout begun
Parts:
- added J1, J10, J11, J12, J13, J14, J15, J16, J17, J18, J19, J2, J20, J21, J22, J23, J24, J25, J3, J4, J5, J6, J7, J8, J9: Conn_01x02_Male, Pin_Headers:Pin_Header_Straight_1x02_Pitch2.54mm, symbol Connector:Conn_01x02_Male
- U1: renamed from U?; footprint (none) -> teensy:Teensy30_31_32_LC
Connections:
- net labels added: +5V, GND, IO_0, IO_1, IO_10, IO_11, IO_12, IO_13, IO_14, IO_15, IO_16, IO_17, IO_18, IO_19, IO_2, IO_20, IO_21, IO_22, IO_23, IO_3, IO_4, IO_5, IO_6, IO_7, IO_8, IO_9, Vin
- wire segments 0 -> 79
- no-connect marks 0 -> 28

Commit message: Updated SCH and PCB to use fewer header footprints
Parts:
- removed J1, J10, J11, J12, J13, J14, J15, J16, J18, J19, J2, J20, J21, J22, J23, J24, J25, J3, J4, J5, J6, J7, J8, J9: Conn_01x02_Male, Pin_Headers:Pin_Header_Straight_1x02_Pitch2.54mm, symbol Connector:Conn_01x02_Male
- added J1, J2, J3, J4: Conn_01x12_Male, Pin_Headers:Pin_Header_Straight_1x12_Pitch2.54mm, symbol Connector:Conn_01x12_Male
- U1: footprint teensy:Teensy30_31_32_LC -> Teensy32NoCenterPads:Teensy30_31_32_LC_NoCenterPads
- renumbered J17 to J5
Connections:
- wire segments 79 -> 82

Commit message: Added I2C, SPI headers, rear Teensy pins
Parts:
- removed J1, J2, J3, J4: Conn_01x12_Male, Pin_Headers:Pin_Header_Straight_1x12_Pitch2.54mm, symbol Connector:Conn_01x12_Male
- added J1, J2, J3, J4: Conn_01x14_Male, Pin_Headers:Pin_Header_Straight_1x14_Pitch2.54mm, symbol Connector:Conn_01x14_Male
- added J5: Conn_01x03_Male, Pin_Headers:Pin_Header_Straight_1x03_Pitch2.54mm, symbol Connector:Conn_01x03_Male
- added J6: Conn_01x05_Male, symbol Connector:Conn_01x05_Male
- U1: footprint Teensy32NoCenterPads:Teensy30_31_32_LC_NoCenterPads -> Teensy32NoCenterPads:Teensy30_31_32_LC_EdgePads
- renumbered J5 to J7
Connections:
- net labels added: 3V3, A14, PROG, VBAT
- wire segments 82 -> 102
- no-connect marks 28 -> 24
Other:
- note added: "GND\nCS\nDOUT\nDIN\nSCK"
- note added: "GND\nDATA\nCLK\n"

Commit message: Added USB cutout, fixed labels.
Parts:
- J6: footprint (none) -> Pin_Headers:Pin_Header_Straight_1x05_Pitch2.54mm
Changed lines of the file:
@@
 F 0 "J6" H 8456 2628 50  0000 C CNN
 F 1 "Conn_01x05_Male" H 8456 2537 50  0000 C CNN
-F 2 "" H 8350 2250 50  0001 C CNN
+F 2 "Pin_Headers:Pin_Header_Straight_1x05_Pitch2.54mm" H 8350 2250 50  0001 C CNN
 F 3 "~" H 8350 2250 50  0001 C CNN
 	1    8350 2250

Commit message: Added 3V3 rail, moved I2C/SPI/VIN headers
Parts:
- added J8, J9: Conn_01x14_Male, Pin_Headers:Pin_Header_Straight_1x14_Pitch2.54mm, symbol Connector:Conn_01x14_Male
Connections:
- wire segments 102 -> 130
Changed lines of the file:
@@
 U 1 1 5BBD8B92
 P 7200 3800
-F 0 "J4" H 7173 3773 50  0000 R CNN
-F 1 "Conn_01x14_Male" H 7173 3682 50  0000 R CNN
+F 0 "J4" H 7150 3850 50  0000 R CNN
+F 1 "Conn_01x14_Male" V 7100 3750 50  0000 R CNN
 F 2 "Pin_Headers:Pin_Header_Straight_1x14_Pitch2.54mm" H 7200 3800 50  0001 C CNN
 F 3 "~" H 7200 3800 50  0001 C CNN
@@
 U 1 1 5BBDA01C
 P 7200 2200
-F 0 "J2" H 7173 2173 50  0000 R CNN
-F 1 "Conn_01x14_Male" H 7173 2082 50  0000 R CNN
+F 0 "J2" H 7150 2250 50  0000 R CNN
+F 1 "Conn_01x14_Male" V 7100 2150 50  0000 R CNN
 F 2 "Pin_Headers:Pin_Header_Straight_1x14_Pitch2.54mm" H 7200 2200 50  0001 C CNN
 F 3 "~" H 7200 2200 50  0001 C CNN
@@
 Wire Wire Line
 	8550 2050 8700 2050
+$Comp
+L Connector:Conn_01x14_Male J8
+U 1 1 5BE253DF
+P 7700 2200
+F 0 "J8" H 7650 2250 50  0000 R CNN
+F 1 "Conn_01x14_Male" V 7600 2150 50  0000 R CNN
+F 2 "Pin_Headers:Pin_Header_Straight_1x14_Pitch2.54mm" H 7700 2200 50  0001 C CNN
+F 3 "~" H 7700 2200 50  0001 C CNN
+	1    7700 2200
+	-1   0    0    -1
+$EndComp
+$Comp
+L Connector:Conn_01x14_Male J9
+U 1 1 5BE25488
+P 7700 3800
+F 0 "J9" H 7650 3850 50  0000 R CNN
+F 1 "Conn_01x14_Male" V 7600 3750 50  0000 R CNN
+F 2 "Pin_Headers:Pin_Header_Straight_1x14_Pitch2.54mm" H 7700 3800 50  0001 C CNN
+F 3 "~" H 7700 3800 50  0001 C CNN
+	1    7700 3800
+	-1   0    0    -1
+$EndComp
+Text GLabel 7500 3050 2    39   Input ~ 0
+3V3
+Text GLabel 7500 1450 2    39   Input ~ 0
+3V3
+Wire Wire Line
+	7500 1450 7500 1600
+Connection ~ 7500 1600
+Wire Wire Line
+	7500 1600 7500 1700
+Connection ~ 7500 1700
+Wire Wire Line
+	7500 1700 7500 1800
+Connection ~ 7500 1800
+Wire Wire Line
+	7500 1800 7500 1900
+Connection ~ 7500 1900
+Wire Wire Line
+	7500 1900 7500 2000
+Connection ~ 7500 2000
+Wire Wire Line
+	7500 2000 7500 2100
+Connection ~ 7500 2100
+Wire Wire Line
+	7500 2100 7500 2200
+Connection ~ 7500 2200
+Wire Wire Line
+	7500 2200 7500 2300
+Connection ~ 7500 2300
+Wire Wire Line
+	7500 2300 7500 2400
+Connection ~ 7500 2400
+Wire Wire Line
+	7500 2400 7500 2500
+Connection ~ 7500 2500
+Wire Wire Line
+	7500 2500 7500 2600
+Connection ~ 7500 2600
+Wire Wire Line
+	7500 2600 7500 2700
+Connection ~ 7500 2700
+Wire Wire Line
+	7500 2700 7500 2800
+Connection ~ 7500 2800
+Wire Wire Line
+	7500 2800 7500 2900
+Wire Wire Line
+	7500 3050 7500 3200
+Connection ~ 7500 3200
+Wire Wire Line
+	7500 3200 7500 3300
+Connection ~ 7500 3300
+Wire Wire Line
+	7500 3300 7500 3400
+Connection ~ 7500 3400
+Wire Wire Line
+	7500 3400 7500 3500
+Connection ~ 7500 3500
+Wire Wire Line
+	7500 3500 7500 3600
+Connection ~ 7500 3600
+Wire Wire Line
+	7500 3600 7500 3700
+Connection ~ 7500 3700
+Wire Wire Line
+	7500 3700 7500 3800
+Connection ~ 7500 3800
+Wire Wire Line
+	7500 3800 7500 3900
+Connection ~ 7500 3900
+Wire Wire Line
+	7500 3900 7500 4000
+Connection ~ 7500 4000
+Wire Wire Line
+	7500 4000 7500 4100
+Connection ~ 7500 4100
+Wire Wire Line
+	7500 4100 7500 4200
+Connection ~ 7500 4200
+Wire Wire Line
+	7500 4200 7500 4300
+Connection ~ 7500 4300
+Wire Wire Line
+	7500 4300 7500 4400
+Connection ~ 7500 4400
+Wire Wire Line
+	7500 4400 7500 4500
 $EndSCHEMATC
